Commit message: Add files via upload
bo_update

File: urdf/hand_e/hand_e.urdf.xacro (robot description, xacro)
@@ -113,8 +113,14 @@
             <limit lower="0" upper="0.035" effort="0" velocity="0" />
         </joint>
+        <link name="${prefix}Tcp"/>
+        <joint name="${prefix}hand_to_tcp" type="fixed">
+            <origin xyz="0 -0.23 0" rpy="1.57 0 0"/>
+            <parent link="${prefix}dummy_gripper_link"/>
+            <child  link="${prefix}Tcp"/>
+        </joint>
       <xacro:finger prefix="${prefix}" parent="${prefix}slider1" stl_name="${finger1_path}" finger_name="finger1"  joint_name="silder1_to_finger1"/>
       <xacro:finger prefix="${prefix}" parent="${prefix}slider2" stl_name="${finger2_path}" finger_name="finger2"  joint_name="silder2_to_finger2"/>
     </xacro:macro>
     <!-- <link name="world"/>
-    <xacro:hande_no_fingers prefix="" finger1_path="/wiring_iema/finger_right.STL" finger2_path="wiring_iema/finger_left.STL" parent="world" /> -->
+    <xacro:hande_no_fingers prefix="" finger1_path="tactile2x6.STL" finger2_path="tactile2x6.STL" parent="world" />  -->
 </robot>

Commit message: modificato urdf effort limits e velocity per simulaizone

File: urdf/hand_e/hand_e.urdf.xacro (robot description, xacro)
@@ -104,5 +104,5 @@
             <child link="${prefix}slider1"/>
             <axis xyz="0 1 0" />
-            <limit lower="0" upper="0.035" effort="0" velocity="0" />
+            <limit lower="0" upper="0.035" effort="10" velocity="10" />
         </joint>
         <joint name="${prefix}bl_to_slider2"  type="prismatic">
@@ -111,5 +111,5 @@
             <child link="${prefix}slider2"/>
             <axis xyz="0 1 0" />
-            <limit lower="0" upper="0.035" effort="0" velocity="0" />
+            <limit lower="0" upper="0.035" effort="10" velocity="10" />
         </joint>
         <link name="${prefix}Tcp"/>
